Commit message: rebuild

File: yc_ws/src/my_ur_driver/my_moveit_config/srdf/my_world.macro.srdf.xacro (robot description, xacro)
@@ -53,116 +53,4 @@
     <disable_collisions link1="${prefix}wrist_1_link" link2="${prefix}wrist_3_link" reason="Never" />
     <disable_collisions link1="${prefix}wrist_2_link" link2="${prefix}wrist_3_link" reason="Adjacent" />
-    <!-- <disable_collisions link1="robotiq_base_link" link2="robotiq_140_base_link" reason="Adjacent gripper links" />
-    <disable_collisions link1="left_inner_finger" link2="left_inner_finger_pad" reason="Finger self-collision" />
-    <disable_collisions link1="right_inner_finger" link2="right_inner_finger_pad" reason="Finger self-collision" />
-    <disable_collisions link1="left_outer_finger" link2="left_outer_finger_pad" reason="Finger self-collision" />
-    <disable_collisions link1="right_outer_finger" link2="right_outer_finger_pad" reason="Finger self-collision" />
-    <disable_collisions link1="left_inner_finger" link2="left_outer_finger" reason="Finger self-collision" />
-    <disable_collisions link1="right_inner_finger" link2="right_outer_finger" reason="Finger self-collision" /> -->
-    <!-- <disable_collisions link1="left_outer_knuckle" link2="right_outer_knuckle" reason="Finger self-collision2" />
-    <disable_collisions link1="left_inner_knuckle" link2="right_inner_knuckle" reason="Finger self-collision4" />
-    <disable_collisions link1="left_inner_finger" link2="right_inner_finger" reason="Finger self-collision3" />
-    <disable_collisions link1="left_outer_finger" link2="right_outer_finger" reason="Finger self-collision5" />
-    <disable_collisions link1="left_inner_finger_pad" link2="right_inner_finger_pad" reason="Finger self-collision" />
-    <disable_collisions link1="left_outer_finger_pad" link2="right_outer_finger_pad" reason="Finger self-collision" />
-    <disable_collisions link1="robotiq_140_base_link" link2="robotiq_base_link" reason="Finger self-collision" /> -->
-    <!-- <disable_collisions link1="${prefix}robotiq_base_link" link2="${prefix}robotiq_140_base_link" reason="Adjacent gripper links" />
-    <disable_collisions link1="${prefix}left_inner_finger" link2="${prefix}left_inner_finger_pad" reason="Finger self-collision" />
-    <disable_collisions link1="${prefix}right_inner_finger" link2="${prefix}right_inner_finger_pad" reason="Finger self-collision" />
-    <disable_collisions link1="${prefix}left_outer_finger" link2="${prefix}left_outer_knuckle" reason="Finger self-collision" />
-    <disable_collisions link1="${prefix}right_inner_knuckle" link2="${prefix}right_outer_knuckle" reason="Finger self-collision" /> -->
-    <!-- <disable_collisions link1="${prefix}left_inner_finger" link2="${prefix}left_outer_finger" reason="Finger self-collision" />
-    <disable_collisions link1="${prefix}right_inner_finger" link2="${prefix}right_outer_finger" reason="Finger self-collision" />
-    <disable_collisions link1="${prefix}left_outer_knuckle" link2="${prefix}right_outer_knuckle" reason="Knuckle self-collision" />
-    <disable_collisions link1="${prefix}left_inner_knuckle" link2="${prefix}right_inner_knuckle" reason="Knuckle self-collision" />
-    <disable_collisions link1="${prefix}left_finger_tip" link2="${prefix}right_finger_tip" reason="Finger tip self-collision" /> -->
-    <!-- <disable_collisions link1="robotiq_base_link" link2="robotiq_140_base_link" reason="Adjacent" />
-    <disable_collisions link1="left_inner_finger" link2="left_inner_finger_pad" reason="Finger self-collision" />
-    <disable_collisions link1="right_inner_finger" link2="right_inner_finger_pad" reason="Finger self-collision" />
-    <disable_collisions link1="left_outer_knuckle" link2="left_outer_finger" reason="Finger self-collision" />
-    <disable_collisions link1="right_outer_knuckle" link2="right_outer_finger" reason="Finger self-collision" />
-    <disable_collisions link1="tool0" link2="robotiq_base_link" reason="Adjacent" />
-    <disable_collisions link1="robotiq_base_link" link2="left_outer_knuckle" reason="Adjacent" />
-    <disable_collisions link1="robotiq_base_link" link2="right_outer_knuckle" reason="Adjacent" />
-    <disable_collisions link1="robotiq_base_link" link2="left_inner_knuckle" reason="Adjacent" />
-    <disable_collisions link1="robotiq_base_link" link2="right_inner_knuckle" reason="Adjacent" />
-    <disable_collisions link1="left_outer_finger" link2="left_inner_finger" reason="Finger self-collision" />
-    <disable_collisions link1="right_outer_finger" link2="right_inner_finger" reason="Finger self-collision" /> -->
-<!-- Base and Gripper Collisions -->
-    <disable_collisions link1="robotiq_base_link" link2="robotiq_140_base_link" reason="Adjacent" />
-    <disable_collisions link1="robotiq_base_link" link2="left_inner_finger" reason="Finger self-collision" />
-    <disable_collisions link1="robotiq_base_link" link2="left_inner_finger_pad" reason="Finger self-collision" />
-    <disable_collisions link1="robotiq_base_link" link2="left_outer_knuckle" reason="Adjacent" />
-    <disable_collisions link1="robotiq_base_link" link2="left_outer_finger" reason="Finger self-collision" />
-    <disable_collisions link1="robotiq_base_link" link2="right_inner_finger" reason="Finger self-collision" />
-    <disable_collisions link1="robotiq_base_link" link2="right_inner_finger_pad" reason="Finger self-collision" />
-    <disable_collisions link1="robotiq_base_link" link2="right_outer_knuckle" reason="Adjacent" />
-    <disable_collisions link1="robotiq_base_link" link2="right_outer_finger" reason="Finger self-collision" />
-    <disable_collisions link1="robotiq_base_link" link2="left_inner_knuckle" reason="Adjacent" />
-    <disable_collisions link1="robotiq_base_link" link2="right_inner_knuckle" reason="Adjacent" />
-    <disable_collisions link1="robotiq_140_base_link" link2="left_inner_finger" reason="Finger self-collision" />
-    <disable_collisions link1="robotiq_140_base_link" link2="left_inner_finger_pad" reason="Finger self-collision" />
-    <disable_collisions link1="robotiq_140_base_link" link2="left_outer_knuckle" reason="Finger self-collision" />
-    <disable_collisions link1="robotiq_140_base_link" link2="left_outer_finger" reason="Finger self-collision" />
-    <disable_collisions link1="robotiq_140_base_link" link2="right_inner_finger" reason="Finger self-collision" />
-    <disable_collisions link1="robotiq_140_base_link" link2="right_inner_finger_pad" reason="Finger self-collision" />
-    <disable_collisions link1="robotiq_140_base_link" link2="right_outer_knuckle" reason="Finger self-collision" />
-    <disable_collisions link1="robotiq_140_base_link" link2="right_outer_finger" reason="Finger self-collision" />
-    <disable_collisions link1="robotiq_140_base_link" link2="left_inner_knuckle" reason="Finger self-collision" />
-    <disable_collisions link1="robotiq_140_base_link" link2="right_inner_knuckle" reason="Finger self-collision" />
-    <disable_collisions link1="left_inner_finger" link2="left_inner_finger_pad" reason="Finger self-collision" />
-    <disable_collisions link1="left_inner_finger" link2="left_outer_knuckle" reason="Finger self-collision" />
-    <disable_collisions link1="left_inner_finger" link2="left_outer_finger" reason="Finger self-collision" />
-    <disable_collisions link1="left_inner_finger" link2="right_inner_finger" reason="Finger self-collision" />
-    <disable_collisions link1="left_inner_finger" link2="right_inner_finger_pad" reason="Finger self-collision" />
-    <disable_collisions link1="left_inner_finger" link2="right_outer_knuckle" reason="Finger self-collision" />
-    <disable_collisions link1="left_inner_finger" link2="right_outer_finger" reason="Finger self-collision" />
-    <disable_collisions link1="left_inner_finger" link2="left_inner_knuckle" reason="Finger self-collision" />
-    <disable_collisions link1="left_inner_finger" link2="right_inner_knuckle" reason="Finger self-collision" />
-    <disable_collisions link1="left_inner_finger_pad" link2="left_outer_knuckle" reason="Finger self-collision" />
-    <disable_collisions link1="left_inner_finger_pad" link2="left_outer_finger" reason="Finger self-collision" />
-    <disable_collisions link1="left_inner_finger_pad" link2="right_inner_finger" reason="Finger self-collision" />
-    <disable_collisions link1="left_inner_finger_pad" link2="right_inner_finger_pad" reason="Finger self-collision" />
-    <disable_collisions link1="left_inner_finger_pad" link2="right_outer_knuckle" reason="Finger self-collision" />
-    <disable_collisions link1="left_inner_finger_pad" link2="right_outer_finger" reason="Finger self-collision" />
-    <disable_collisions link1="left_inner_finger_pad" link2="left_inner_knuckle" reason="Finger self-collision" />
-    <disable_collisions link1="left_inner_finger_pad" link2="right_inner_knuckle" reason="Finger self-collision" />
-    <disable_collisions link1="left_outer_knuckle" link2="left_outer_finger" reason="Finger self-collision" />
-    <disable_collisions link1="left_outer_knuckle" link2="right_inner_finger" reason="Finger self-collision" />
-    <disable_collisions link1="left_outer_knuckle" link2="right_inner_finger_pad" reason="Finger self-collision" />
-    <disable_collisions link1="left_outer_knuckle" link2="right_outer_knuckle" reason="Finger self-collision" />
-    <disable_collisions link1="left_outer_knuckle" link2="right_outer_finger" reason="Finger self-collision" />
-    <disable_collisions link1="left_outer_knuckle" link2="left_inner_knuckle" reason="Finger self-collision" />
-    <disable_collisions link1="left_outer_knuckle" link2="right_inner_knuckle" reason="Finger self-collision" />
-    <disable_collisions link1="left_outer_finger" link2="right_inner_finger" reason="Finger self-collision" />
-    <disable_collisions link1="left_outer_finger" link2="right_inner_finger_pad" reason="Finger self-collision" />
-    <disable_collisions link1="left_outer_finger" link2="right_outer_knuckle" reason="Finger self-collision" />
-    <disable_collisions link1="left_outer_finger" link2="right_outer_finger" reason="Finger self-collision" />
-    <disable_collisions link1="left_outer_finger" link2="left_inner_knuckle" reason="Finger self-collision" />
-    <disable_collisions link1="left_outer_finger" link2="right_inner_knuckle" reason="Finger self-collision" />
-    <disable_collisions link1="right_inner_finger" link2="right_inner_finger_pad" reason="Finger self-collision" />
-    <disable_collisions link1="right_inner_finger" link2="right_outer_knuckle" reason="Finger self-collision" />
-    <disable_collisions link1="right_inner_finger" link2="right_outer_finger" reason="Finger self-collision" />
-    <disable_collisions link1="right_inner_finger" link2="left_inner_knuckle" reason="Finger self-collision" />
-    <disable_collisions link1="right_inner_finger" link2="right_inner_knuckle" reason="Finger self-collision" />
-    <disable_collisions link1="right_inner_finger_pad" link2="right_outer_knuckle" reason="Finger self-collision" />
-    <disable_collisions link1="right_inner_finger_pad" link2="right_outer_finger" reason="Finger self-collision" />
-    <disable_collisions link1="right_inner_finger_pad" link2="left_inner_knuckle" reason="Finger self-collision" />
-    <disable_collisions link1="right_inner_finger_pad" link2="right_inner_knuckle" reason="Finger self-collision" />
-    <disable_collisions link1="right_outer_knuckle" link2="right_outer_finger" reason="Finger self-collision" />
-    <disable_collisions link1="right_outer_knuckle" link2="left_inner_knuckle" reason="Finger self-collision" />
-    <disable_collisions link1="right_outer_knuckle" link2="right_inner_knuckle" reason="Finger self-collision" />
-    <disable_collisions link1="right_outer_finger" link2="left_inner_knuckle" reason="Finger self-collision" />
-    <disable_collisions link1="right_outer_finger" link2="right_inner_knuckle" reason="Finger self-collision" />
-    <disable_collisions link1="left_inner_knuckle" link2="right_inner_knuckle" reason="Finger self-collision" />
-    <disable_collisions link1="robotiq_base_link" link2="robotiq_140_base_link" reason="Adjacent" />
-    <disable_collisions link1="robotiq_base_link" link2="tool0" reason="Adjacent" />
-    <disable_collisions link1="robotiq_base_link" link2="wrist_1_link" reason="Adjacent" />
-    <disable_collisions link1="robotiq_base_link" link2="wrist_2_link" reason="Adjacent" />
-    <disable_collisions link1="robotiq_base_link" link2="wrist_3_link" reason="Adjacent" />
-    <disable_collisions link1="robotiq_140_base_link" link2="tool0" reason="Adjacent" />
-    <disable_collisions link1="robotiq_140_base_link" link2="wrist_1_link" reason="Adjacent" />
-    <disable_collisions link1="robotiq_140_base_link" link2="wrist_2_link" reason="Adjacent" />
-    <disable_collisions link1="robotiq_140_base_link" link2="wrist_3_link" reason="Adjacent" />
     <disable_collisions link1="tool0" link2="wrist_1_link" reason="Adjacent" />
     <disable_collisions link1="tool0" link2="wrist_2_link" reason="Adjacent" />
@@ -171,18 +59,4 @@
     <disable_collisions link1="wrist_1_link" link2="wrist_3_link" reason="Adjacent" />
     <disable_collisions link1="wrist_2_link" link2="wrist_3_link" reason="Adjacent" />
-    <disable_collisions link1="cam_holder_with_onrobot_single" link2="robotiq_base_link" reason="Adjacent" />
-    <disable_collisions link1="cam_holder_with_onrobot_single" link2="robotiq_140_base_link" reason="Adjacent" />
-    <disable_collisions link1="cam_holder_with_onrobot_single" link2="tool0" reason="Adjacent" />
-    <disable_collisions link1="cam_holder_with_onrobot_single" link2="wrist_1_link" reason="Adjacent" />
-    <disable_collisions link1="cam_holder_with_onrobot_single" link2="wrist_2_link" reason="Adjacent" />
-    <disable_collisions link1="cam_holder_with_onrobot_single" link2="wrist_3_link" reason="Adjacent" />
-    <!-- <disable_collisions link1="tool0_2_cam_holder_with_onrobot_single" link2="robotiq_base_link" reason="Adjacent" />
-    <disable_collisions link1="tool0_2_cam_holder_with_onrobot_single" link2="robotiq_140_base_link" reason="Adjacent" />
-    <disable_collisions link1="tool0_2_cam_holder_with_onrobot_single" link2="tool0" reason="Adjacent" />
-    <disable_collisions link1="tool0_2_cam_holder_with_onrobot_single" link2="wrist_1_link" reason="Adjacent" />
-    <disable_collisions link1="tool0_2_cam_holder_with_onrobot_single" link2="wrist_2_link" reason="Adjacent" />
-    <disable_collisions link1="tool0_2_cam_holder_with_onrobot_single" link2="wrist_3_link" reason="Adjacent" />
- -->
-cam_holder_with_onrobot_single
   </xacro:macro>
 </robot>

File: yc_ws/src/my_ur_driver/my_ur_config/urdf/my_world_with_gripper.urdf.xacro (robot description, xacro)
@@ -5,4 +5,8 @@
    <!-- import main macro -->
    <xacro:include filename="$(find ur_description)/urdf/ur_macro.xacro"/>
+   <xacro:include filename="$(find my_ur_driver)/my_ur_config/urdf/gripper/robotiq_2f_140.xacro" />
+   <xacro:include filename="$(find my_ur_driver)/my_ur_config/urdf/gripper/robotiq_2f_140_gripper.urdf.xacro" />
+   <xacro:include filename="$(find my_ur_driver)/my_ur_config/urdf/gripper/2f_140.ros2_control.xacro" />
+   <xacro:include filename="$(find my_ur_driver)/my_ur_config/urdf/gripper/ur_to_robotiq_adapter.urdf.xacro" />
    <!-- possible 'ur_type' values: ur3, ur3e, ur5, ur5e, ur10, ur10e, ur16e, ur20, ur30 -->
    <!-- the default value should raise an error in case this was called without defining the type -->
@@ -51,4 +55,34 @@
    <!-- create link fixed to the "world" -->
    <link name="world" />
+  <!-- for onrobot straight mode -->
+    <!-- 10mm cam_holder_thickness, 13mm quick change adapter thickness, xxmm from vgc10 base to suction tip-->
+      <link name="cam_holder_with_onrobot_single">
+      <inertial>
+        <origin xyz="0.00010121 -0.030402 0.046358" rpy="0 0 0" />
+        <!-- <origin xyz=".00121 -0.030402 0.046358" rpy="0 0 0" /> -->
+        <mass value="0.6381" />
+        <inertia ixx="0.00053122" ixy="-4.1332E-09" ixz="3.2568E-07" iyy="0.00043426" iyz="-1.2224E-05" izz="0.00056022" />
+      </inertial>
+      <visual>
+        <origin xyz="0 0 0" rpy="0 0 0" />
+        <geometry>
+          <mesh filename="package://my_ur_driver/my_ur_config/urdf/meshes/camera/abdo_camera.stl" />
+        </geometry>
+        <material name="">
+          <color rgba="0.79216 0.81961 0.93333 1" />
+        </material>
+      </visual>
+      <collision>
+        <origin xyz="0 0 0" rpy="0 0 0" />
+        <geometry>
+          <mesh filename="package://my_ur_driver/my_ur_config/urdf/meshes/camera/abdo_camera.stl" />
+        </geometry>
+      </collision>
+    </link>
+    <joint name="tool0_2_cam_holder_with_onrobot_single" type="fixed">
+      <parent link="tool0" />
+      <child link="cam_holder_with_onrobot_single" />
+      <origin xyz="0 0 0" rpy="0 0 0" />
+    </joint>
    <!-- arm -->
    <xacro:ur_robot
@@ -112,52 +146,9 @@
     </gazebo>
   </xacro:if>
- <!-- for onrobot straight mode -->
-  <!-- 10mm cam_holder_thickness, 13mm quick change adapter thickness, xxmm from vgc10 base to suction tip-->
-  <link name="tcp_vgc10" />
-  <joint name="tool0_2_tcp_vgc10" type="fixed">
+  <!-- <joint name="robotiq_2f_140_fixed" type="fixed">
     <parent link="tool0" />
-    <child link="tcp_vgc10" />
-    <!-- <origin xyz="0 0 0.180" rpy="0 0 0" />   -->
-    <origin xyz="0 0 0.175" rpy="0 0 0" />
-    <!-- unverified values -->
-  </joint>
-  <!-- for onrobot straight mode -->
-  <!-- 10mm cam_holder_thickness, 13mm quick change adapter thickness, 200mm from rg2 base to a logical finger pick point (not the extreme finger tip) -->
-  <link name="tcp_rg2" />
-  <joint name="tool0_2_tcp_rg2" type="fixed">
-    <parent link="tool0" />
-    <child link="tcp_rg2" />
-    <!-- <origin xyz="0 0 0.223" rpy="0 0 0" /> -->
-    <!-- <origin xyz="0 0 0.235" rpy="0 0 0" /> -->
-    <origin xyz="0 0 0.232" rpy="0 0 0" />
-  </joint>
-    <link name="cam_holder_with_onrobot_single">
-    <inertial>
-      <origin xyz="0.00010121 -0.030402 0.046358" rpy="0 0 0" />
-      <!-- <origin xyz=".00121 -0.030402 0.046358" rpy="0 0 0" /> -->
-      <mass value="0.6381" />
-      <inertia ixx="0.00053122" ixy="-4.1332E-09" ixz="3.2568E-07" iyy="0.00043426" iyz="-1.2224E-05" izz="0.00056022" />
-    </inertial>
-    <visual>
-      <origin xyz="0 0 0" rpy="0 0 0" />
-      <geometry>
-        <mesh filename="package://my_ur_driver/my_ur_conifg/urdf/meshes/camera/abdo_camera.stl" />
-      </geometry>
-      <material name="">
-        <color rgba="0.79216 0.81961 0.93333 1" />
-      </material>
-    </visual>
-    <collision>
-      <origin xyz="0 0 0" rpy="0 0 0" />
-      <geometry>
-        <mesh filename="package://my_ur_driver/my_ur_conifgurdf/meshes/camera/abdo_camera.stl" />
-      </geometry>
-    </collision>
-  </link>
-  <joint name="tool0_2_cam_holder_with_onrobot_single" type="fixed">
-    <parent link="tool0" />
-    <child link="cam_holder_with_onrobot_single" />
-    <origin xyz="0 0 0" rpy="0 0 0" />
-  </joint>
+    <child link="robotiq_2f_140" />
+    <origin xyz="0 0 0.205" rpy="0 0 0" />
+  </joint> -->
     <!-- this part deals with the tcp end effector transform, not related to the visual/collision. -->
   <!-- so far tcp_gripper is always required even if u dun use it, because the my_robot_advance.cpp always look for it at the start -->
