Commit message: Update record and gazebo

File: yc_ws/src/my_ur_driver/my_ur_config/urdf/my_world.urdf.xacro (robot description, xacro)
@@ -142,5 +142,5 @@
       <origin xyz="0 0 0" rpy="0 0 0" />
       <geometry>
-        <mesh filename="package://my_ur_driver/my_ur_conifg/urdf/meshes/camera/abdo_camera.stl" />
+        <mesh filename="package://my_ur_driver/my_ur_config/urdf/meshes/camera/abdo_camera.stl" />
       </geometry>
       <material name="">
@@ -151,5 +151,5 @@
       <origin xyz="0 0 0" rpy="0 0 0" />
       <geometry>
-        <mesh filename="package://my_ur_driver/my_ur_conifgurdf/meshes/camera/abdo_camera.stl" />
+        <mesh filename="package://my_ur_driver/my_ur_config/urdf/meshes/camera/abdo_camera.stl" />
       </geometry>
     </collision>
